Commit message: feat: 为小车添加 6-DOF 机械臂并增大底盘
- 新增 arm.urdf.xacro：7 连杆 6 旋转关节（基座旋转/肩/肘/腕滚转/腕俯仰/末端旋转）
- 底盘增大：radius 0.10->0.14, length 0.12->0.16, 质量 1.0->2.5kg（惯量同步更新）
- 轮距 0.20->0.28，轮子/caster/激光/摄像头位置随底盘调整
- ros2_control 添加 6 个机械臂关节 position 接口
- 新增 arm_controller（joint_trajectory_controller）并在 launch 中加载
- nav2 robot_radius 0.12->0.16

File: src/fishbot_description/urdf/fishbot/base.urdf.xacro (robot description, xacro)
@@ -2,5 +2,5 @@
 <robot xmlns:xacro = "http://www.ros.org/wiki/xacro">
     <xacro:include filename="$(find fishbot_description)/urdf/fishbot/common_inertia.xacro"/>
-    <xacro:macro name = "base_xacro" params = "length radius">
+    <xacro:macro name = "base_xacro" params = "length radius mass">
         <link name="base_footprint"/>
         <!-- 机器人身体部分 -->
@@ -25,5 +25,5 @@
                 </material>
             </collision>
-            <xacro:cylinder_inertia m="1.0" r="${radius}" h="${length}" />
+            <xacro:cylinder_inertia m="${mass}" r="${radius}" h="${length}" />
         </link>
         <joint name="joint_name" type="fixed">

File: src/fishbot_description/urdf/fishbot/fishbot.ros2_control.xacro (robot description, xacro)
@@ -32,4 +32,59 @@
                     <state_interface name="effort" />
                 </joint>
+                <!-- ============ 六自由度机械臂关节 ============ -->
+                <joint name="arm_joint1">
+                    <command_interface name="position">
+                        <param name="min">-3.14159</param>
+                        <param name="max">3.14159</param>
+                    </command_interface>
+                    <state_interface name="position" />
+                    <state_interface name="velocity" />
+                    <state_interface name="effort" />
+                </joint>
+                <joint name="arm_joint2">
+                    <command_interface name="position">
+                        <param name="min">-2.0</param>
+                        <param name="max">2.0</param>
+                    </command_interface>
+                    <state_interface name="position" />
+                    <state_interface name="velocity" />
+                    <state_interface name="effort" />
+                </joint>
+                <joint name="arm_joint3">
+                    <command_interface name="position">
+                        <param name="min">-2.5</param>
+                        <param name="max">1.5</param>
+                    </command_interface>
+                    <state_interface name="position" />
+                    <state_interface name="velocity" />
+                    <state_interface name="effort" />
+                </joint>
+                <joint name="arm_joint4">
+                    <command_interface name="position">
+                        <param name="min">-3.14159</param>
+                        <param name="max">3.14159</param>
+                    </command_interface>
+                    <state_interface name="position" />
+                    <state_interface name="velocity" />
+                    <state_interface name="effort" />
+                </joint>
+                <joint name="arm_joint5">
+                    <command_interface name="position">
+                        <param name="min">-2.0</param>
+                        <param name="max">2.0</param>
+                    </command_interface>
+                    <state_interface name="position" />
+                    <state_interface name="velocity" />
+                    <state_interface name="effort" />
+                </joint>
+                <joint name="arm_joint6">
+                    <command_interface name="position">
+                        <param name="min">-3.14159</param>
+                        <param name="max">3.14159</param>
+                    </command_interface>
+                    <state_interface name="position" />
+                    <state_interface name="velocity" />
+                    <state_interface name="effort" />
+                </joint>
             </ros2_control>
         <gazebo>

File: src/fishbot_description/urdf/fishbot/fishbot.urdf.xacro (robot description, xacro)
@@ -10,16 +10,25 @@
 <xacro:include filename="$(find fishbot_description)/urdf/fishbot/actuator/wheel.urdf.xacro"/>
 <xacro:include filename="$(find fishbot_description)/urdf/fishbot/actuator/caster.urdf.xacro"/>
+<!-- 六自由度机械臂 -->
+<xacro:include filename="$(find fishbot_description)/urdf/fishbot/actuator/arm.urdf.xacro"/>
 <!-- 插件 -->
 <!-- <xacro:include filename="$(find fishbot_description)/urdf/fishbot/plugins/gazebo_control_plugin.xacro"/> -->
 <xacro:include filename="$(find fishbot_description)/urdf/fishbot/plugins/gazebo_sensor_plugin.xacro"/>
 <xacro:include filename="$(find fishbot_description)/urdf/fishbot/fishbot.ros2_control.xacro"/>
-<xacro:base_xacro length = "0.12" radius = "0.10"/>
+<!-- 底盘：为承载机械臂，体积由 r=0.10/h=0.12 增大至 r=0.14/h=0.16，质量 1.0 -> 2.5 kg -->
+<xacro:base_xacro length = "0.16" radius = "0.14" mass = "2.5"/>
 <xacro:imu_xacro xyz="0.0 0.0 0.02"/>
-<xacro:camera_xacro xyz="0.10 0.0 0.075"/>
-<xacro:laser_xacro xyz="0.0 0.0 0.10"/>
-<xacro:wheel_xacro wheel_name = "left_wheel" xyz="0.0 0.10 -0.06"/>
-<xacro:wheel_xacro wheel_name = "right_wheel" xyz="0.0 -0.10 -0.06"/>
-<xacro:caster_xacro caster_name = "front_caster" xyz = "0.08 0.0 -0.076"/>
-<xacro:caster_xacro caster_name = "back_caster" xyz = "-0.08 0.0 -0.076"/>
+<!-- 摄像头前移至 x=0.12，给机械臂基座留出顶部空间 -->
+<xacro:camera_xacro xyz="0.12 0.0 0.075"/>
+<!-- 激光雷达后移至 x=-0.06，与顶部中央的机械臂错开 -->
+<xacro:laser_xacro xyz="-0.06 0.0 0.10"/>
+<!-- 轮距随底盘半径增大：y=±0.14（原 ±0.10），z 下移至 -0.08 保持触地 -->
+<xacro:wheel_xacro wheel_name = "left_wheel" xyz="0.0 0.14 -0.08"/>
+<xacro:wheel_xacro wheel_name = "right_wheel" xyz="0.0 -0.14 -0.08"/>
+<!-- 万向轮外移并下移，保持支撑稳定 -->
+<xacro:caster_xacro caster_name = "front_caster" xyz = "0.10 0.0 -0.096"/>
+<xacro:caster_xacro caster_name = "back_caster" xyz = "-0.10 0.0 -0.096"/>
+<!-- 六自由度机械臂实例化 -->
+<xacro:arm_xacro/>
 <!-- <xacro:gazebo_control_plugin /> -->
 <xacro:gazebo_sensor_plugin/>
