Commit message: feat: 小车改为四轮长方体底盘 + 集成开源 Franka Panda 七自由度机械臂
- 新增 src/panda_description 包（moveit_resources 开源 Panda 描述，含官方 mesh/惯量/限位）
- 底盘：圆柱 -> 长方体 0.70×0.50×0.22 m（质量 8kg），2轮+万向轮 -> 四轮驱动（r=0.05, 轮距0.48）
- ros2_control：4 轮 velocity + Panda 7 关节 position；diff_drive wheels_per_side=2
- MoveIt：SRDF（7 关节 + 官方碰撞豁免）、joint_limits（Panda 限位）、控制器映射更新
- launch：修复并发 spawn 崩溃（TimerAction 延迟 + world 参数可覆盖）
- MuJoCo：同步更新为四轮底盘 + Panda（STL mesh + 官方惯量）
- README 同步更新

File: src/fishbot_description/urdf/fishbot/actuator/wheel.urdf.xacro (robot description, xacro)
@@ -10,5 +10,5 @@
                 <geometry>
                 <!-- 单位：m -->
-                    <cylinder radius="0.032" length="0.04"/>
+                    <cylinder radius="0.05" length="0.04"/>
                 </geometry>
                 <material name="yellow">
@@ -20,5 +20,5 @@
                 <geometry>
                 <!-- 单位：m -->
-                    <cylinder radius="0.032" length="0.04"/>
+                    <cylinder radius="0.05" length="0.04"/>
                 </geometry>
                 <material name="yellow">
@@ -26,5 +26,5 @@
                 </material>
             </collision>
-            <xacro:cylinder_inertia m="0.05" r="0.032" h="0.04"/>
+            <xacro:cylinder_inertia m="0.3" r="0.05" h="0.04"/>
         </link>
         <!-- 机器人关节，用于组合机器人部件 -->

File: src/fishbot_description/urdf/fishbot/base.urdf.xacro (robot description, xacro)
@@ -2,13 +2,13 @@
 <robot xmlns:xacro = "http://www.ros.org/wiki/xacro">
     <xacro:include filename="$(find fishbot_description)/urdf/fishbot/common_inertia.xacro"/>
-    <xacro:macro name = "base_xacro" params = "length radius mass">
+    <!-- 四轮长方体底盘：length(x) × width(y) × height(z)，质量 mass -->
+    <xacro:macro name = "base_xacro" params = "length width height mass">
         <link name="base_footprint"/>
         <!-- 机器人身体部分 -->
         <link name="base_link">
-            <!-- 部件的外观 -->
             <visual>
                 <origin xyz="0.0 0.0 0.0" rpy="0.0 0.0 0.0"/>
                 <geometry>
-                    <cylinder radius="${radius}" length="${length}"/>
+                    <box size="${length} ${width} ${height}"/>
                 </geometry>
                 <material name="white">
@@ -19,5 +19,5 @@
                 <origin xyz="0.0 0.0 0.0" rpy="0.0 0.0 0.0"/>
                 <geometry>
-                    <cylinder radius="${radius}" length="${length}"/>
+                    <box size="${length} ${width} ${height}"/>
                 </geometry>
                 <material name="white">
@@ -25,8 +25,10 @@
                 </material>
             </collision>
-            <xacro:cylinder_inertia m="${mass}" r="${radius}" h="${length}" />
+            <!-- 长方体惯量：ixx∝y²+z², iyy∝x²+z², izz∝x²+y² -->
+            <xacro:box_inertia m="${mass}" w="${length}" h="${width}" d="${height}"/>
         </link>
+        <!-- base_footprint -> base_link：中心在地面上方 height/2 -->
         <joint name="joint_name" type="fixed">
-            <origin xyz="0.0 0.0 ${length/2.0 + 0.032-0.001}" rpy="0.0 0.0 0.0"/>
+            <origin xyz="0.0 0.0 ${height/2.0}" rpy="0.0 0.0 0.0"/>
             <parent link="base_footprint"/>
             <child link="base_link"/>
@@ -34,3 +36,2 @@
     </xacro:macro>
 </robot>
-<!-- 6.3.1 -->

File: src/fishbot_description/urdf/fishbot/fishbot.ros2_control.xacro (robot description, xacro)
@@ -6,12 +6,13 @@
                     <plugin>gazebo_ros2_control/GazeboSystem</plugin>
                 </hardware>
-                <joint name="left_wheel_joint">
+                <!-- ============ 四轮驱动（差速） ============ -->
+                <joint name="left_front_wheel_joint">
                     <command_interface name="velocity">
-                        <param name="min">-1</param>
-                        <param name="max">1</param>
+                        <param name="min">-2</param>
+                        <param name="max">2</param>
                     </command_interface>
                     <command_interface name="effort">
-                        <param name="min">-0.1</param>
-                        <param name="max">0.1</param>
+                        <param name="min">-5</param>
+                        <param name="max">5</param>
                     </command_interface>
                     <state_interface name="position" />
@@ -19,12 +20,12 @@
                     <state_interface name="effort" />
                 </joint>
-                <joint name="right_wheel_joint">
+                <joint name="left_back_wheel_joint">
                     <command_interface name="velocity">
-                        <param name="min">-1</param>
-                        <param name="max">1</param>
+                        <param name="min">-2</param>
+                        <param name="max">2</param>
                     </command_interface>
                     <command_interface name="effort">
-                        <param name="min">-0.1</param>
-                        <param name="max">0.1</param>
+                        <param name="min">-5</param>
+                        <param name="max">5</param>
                     </command_interface>
                     <state_interface name="position" />
@@ -32,9 +33,12 @@
                     <state_interface name="effort" />
                 </joint>
-                <!-- ============ 六自由度机械臂关节 ============ -->
-                <joint name="arm_joint1">
-                    <command_interface name="position">
-                        <param name="min">-3.14159</param>
-                        <param name="max">3.14159</param>
+                <joint name="right_front_wheel_joint">
+                    <command_interface name="velocity">
+                        <param name="min">-2</param>
+                        <param name="max">2</param>
+                    </command_interface>
+                    <command_interface name="effort">
+                        <param name="min">-5</param>
+                        <param name="max">5</param>
                     </command_interface>
                     <state_interface name="position" />
@@ -42,8 +46,12 @@
                     <state_interface name="effort" />
                 </joint>
-                <joint name="arm_joint2">
-                    <command_interface name="position">
-                        <param name="min">-2.0</param>
-                        <param name="max">2.0</param>
+                <joint name="right_back_wheel_joint">
+                    <command_interface name="velocity">
+                        <param name="min">-2</param>
+                        <param name="max">2</param>
+                    </command_interface>
+                    <command_interface name="effort">
+                        <param name="min">-5</param>
+                        <param name="max">5</param>
                     </command_interface>
                     <state_interface name="position" />
@@ -51,8 +59,9 @@
                     <state_interface name="effort" />
                 </joint>
-                <joint name="arm_joint3">
+                <!-- ============ Franka Panda 七自由度机械臂 ============ -->
+                <joint name="panda_joint1">
                     <command_interface name="position">
-                        <param name="min">-2.5</param>
-                        <param name="max">1.5</param>
+                        <param name="min">-2.9671</param>
+                        <param name="max">2.9671</param>
                     </command_interface>
                     <state_interface name="position" />
@@ -60,8 +69,8 @@
                     <state_interface name="effort" />
                 </joint>
-                <joint name="arm_joint4">
+                <joint name="panda_joint2">
                     <command_interface name="position">
-                        <param name="min">-3.14159</param>
-                        <param name="max">3.14159</param>
+                        <param name="min">-1.8326</param>
+                        <param name="max">1.8326</param>
                     </command_interface>
                     <state_interface name="position" />
@@ -69,8 +78,8 @@
                     <state_interface name="effort" />
                 </joint>
-                <joint name="arm_joint5">
+                <joint name="panda_joint3">
                     <command_interface name="position">
-                        <param name="min">-2.0</param>
-                        <param name="max">2.0</param>
+                        <param name="min">-2.9671</param>
+                        <param name="max">2.9671</param>
                     </command_interface>
                     <state_interface name="position" />
@@ -78,8 +87,54 @@
                     <state_interface name="effort" />
                 </joint>
-                <joint name="arm_joint6">
+                <joint name="panda_joint4">
                     <command_interface name="position">
-                        <param name="min">-3.14159</param>
-                        <param name="max">3.14159</param>
+                        <param name="min">-3.0543</param>
+                        <param name="max">3.0543</param>
+                    </command_interface>
+                    <state_interface name="position" />
+                    <state_interface name="velocity" />
+                    <state_interface name="effort" />
+                </joint>
+                <joint name="panda_joint5">
+                    <command_interface name="position">
+                        <param name="min">-2.9671</param>
+                        <param name="max">2.9671</param>
+                    </command_interface>
+                    <state_interface name="position" />
+                    <state_interface name="velocity" />
+                    <state_interface name="effort" />
+                </joint>
+                <joint name="panda_joint6">
+                    <command_interface name="position">
+                        <param name="min">-0.0873</param>
+                        <param name="max">3.8223</param>
+                    </command_interface>
+                    <state_interface name="position" />
+                    <state_interface name="velocity" />
+                    <state_interface name="effort" />
+                </joint>
+                <joint name="panda_joint7">
+                    <command_interface name="position">
+                        <param name="min">-2.9671</param>
+                        <param name="max">2.9671</param>
+                    </command_interface>
+                    <state_interface name="position" />
+                    <state_interface name="velocity" />
+                    <state_interface name="effort" />
+                </joint>
+                <!-- Panda 手爪（可选控制） -->
+                <joint name="panda_finger_joint1">
+                    <command_interface name="position">
+                        <param name="min">0.0</param>
+                        <param name="max">0.04</param>
+                    </command_interface>
+                    <state_interface name="position" />
+                    <state_interface name="velocity" />
+                    <state_interface name="effort" />
+                </joint>
+                <joint name="panda_finger_joint2">
+                    <command_interface name="position">
+                        <param name="min">0.0</param>
+                        <param name="max">0.04</param>
                     </command_interface>
                     <state_interface name="position" />

File: src/fishbot_description/urdf/fishbot/fishbot.urdf.xacro (robot description, xacro)
@@ -1,5 +1,5 @@
 <?xml version="1.0"?>
 <robot xmlns:xacro = "http://www.ros.org/wiki/xacro" name="fishbot">
-<!-- 基础部分 base_link -->
+<!-- 基础部分 base_link（四轮长方体底盘） -->
 <xacro:include filename="$(find fishbot_description)/urdf/fishbot/base.urdf.xacro"/>
 <!-- 传感器部分 -->
@@ -7,29 +7,36 @@
 <xacro:include filename="$(find fishbot_description)/urdf/fishbot/sensor/laser.urdf.xacro"/>
 <xacro:include filename="$(find fishbot_description)/urdf/fishbot/sensor/camera.urdf.xacro"/>
-<!-- 执行器部分 -->
+<!-- 执行器部分：四轮 -->
 <xacro:include filename="$(find fishbot_description)/urdf/fishbot/actuator/wheel.urdf.xacro"/>
-<xacro:include filename="$(find fishbot_description)/urdf/fishbot/actuator/caster.urdf.xacro"/>
-<!-- 六自由度机械臂 -->
-<xacro:include filename="$(find fishbot_description)/urdf/fishbot/actuator/arm.urdf.xacro"/>
+<!-- Franka Emika Panda 七自由度机械臂（开源描述，位于 panda_description 包） -->
+<xacro:include filename="$(find panda_description)/urdf/panda.urdf.xacro"/>
 <!-- 插件 -->
-<!-- <xacro:include filename="$(find fishbot_description)/urdf/fishbot/plugins/gazebo_control_plugin.xacro"/> -->
 <xacro:include filename="$(find fishbot_description)/urdf/fishbot/plugins/gazebo_sensor_plugin.xacro"/>
 <xacro:include filename="$(find fishbot_description)/urdf/fishbot/fishbot.ros2_control.xacro"/>
-<!-- 底盘：为承载机械臂，体积由 r=0.10/h=0.12 增大至 r=0.14/h=0.16，质量 1.0 -> 2.5 kg -->
-<xacro:base_xacro length = "0.16" radius = "0.14" mass = "2.5"/>
-<xacro:imu_xacro xyz="0.0 0.0 0.02"/>
-<!-- 摄像头前移至 x=0.12，给机械臂基座留出顶部空间 -->
-<xacro:camera_xacro xyz="0.12 0.0 0.075"/>
-<!-- 激光雷达后移至 x=-0.06，与顶部中央的机械臂错开 -->
-<xacro:laser_xacro xyz="-0.06 0.0 0.10"/>
-<!-- 轮距随底盘半径增大：y=±0.14（原 ±0.10），z 下移至 -0.08 保持触地 -->
-<xacro:wheel_xacro wheel_name = "left_wheel" xyz="0.0 0.14 -0.08"/>
-<xacro:wheel_xacro wheel_name = "right_wheel" xyz="0.0 -0.14 -0.08"/>
-<!-- 万向轮外移并下移，保持支撑稳定 -->
-<xacro:caster_xacro caster_name = "front_caster" xyz = "0.10 0.0 -0.096"/>
-<xacro:caster_xacro caster_name = "back_caster" xyz = "-0.10 0.0 -0.096"/>
-<!-- 六自由度机械臂实例化 -->
-<xacro:arm_xacro/>
-<!-- <xacro:gazebo_control_plugin /> -->
+<!-- ================= 底盘：四轮长方体 =================
+     尺寸按 Panda 机械臂（总重约 18kg，臂展 0.855m）设计：
+     长 0.70 × 宽 0.50 × 高 0.22 m，质量 8 kg（保证承载稳定）
+     base_footprint 在地面，base_link 中心在 z=0.11 -->
+<xacro:base_xacro length = "0.70" width = "0.50" height = "0.22" mass = "8.0"/>
+<!-- 传感器位置（Panda 占据顶部中央，激光后移、相机前移） -->
+<xacro:imu_xacro xyz="0.0 0.0 0.05"/>
+<xacro:camera_xacro xyz="0.28 0.0 0.05"/>
+<xacro:laser_xacro xyz="-0.12 0.0 0.16"/>
+<!-- 四轮：前左/前右/后左/后右
+     轮子半径 0.05，中心 y=±0.24（外露于 0.25 半宽），x=±0.20（轴距 0.40），z=-0.06（着地） -->
+<xacro:wheel_xacro wheel_name = "left_front_wheel" xyz="0.20 0.24 -0.06"/>
+<xacro:wheel_xacro wheel_name = "left_back_wheel"  xyz="-0.20 0.24 -0.06"/>
+<xacro:wheel_xacro wheel_name = "right_front_wheel" xyz="0.20 -0.24 -0.06"/>
+<xacro:wheel_xacro wheel_name = "right_back_wheel"  xyz="-0.20 -0.24 -0.06"/>
+<!-- ================= Franka Panda 机械臂 =================
+     安装在底盘顶面中央：base_link 顶面 z=0.11 -->
+<joint name="panda_base_joint" type="fixed">
+    <origin xyz="0.0 0.0 0.11" rpy="0.0 0.0 0.0"/>
+    <parent link="base_link"/>
+    <child link="panda_link0"/>
+</joint>
+<gazebo reference="base_link">
+    <selfCollide>false</selfCollide>
+</gazebo>
 <xacro:gazebo_sensor_plugin/>
 <xacro:fishbot_ros2_control/>
